File: VGA-card/KiCAD/AppleVGA.kicad_pcb (KiCad board)
At the start: 2 copper layers, 172.7 x 69.1 mm, 34 parts, among them J1 AppleIIBus, J2 VGA, J3 VGA, SW1 SW_Push, U1 74LVC245, U2 74LVC245, U3 74LVC245, U4 74LS07, U5 UA78M33CKCS, U6 Pico

Commit message: KiCAD error fixes
Connections:
- net +3V3 renamed +3.3V
- J1 pad 1: /Connections/~{IOSEL} -> unconnected-(J1-Pad1)
- J1 pad 19: /Connections/SYNC -> unconnected-(J1-Pad19)
- J1 pad 20: /Connections/~{IOSTRB} -> unconnected-(J1-Pad20)
- J1 pad 21: /Connections/~{RDY} -> unconnected-(J1-Pad21)
- J1 pad 22: /Connections/~{DMA} -> unconnected-(J1-Pad22)
- J1 pad 29: /Connections/~{NMI} -> unconnected-(J1-Pad29)
- J1 pad 30: /Connections/~{IRQ} -> unconnected-(J1-Pad30)
- J1 pad 31: /Connections/~{RES} -> unconnected-(J1-Pad31)
- J1 pad 32: /Connections/~{INH} -> unconnected-(J1-Pad32)
- J1 pad 36: /Connections/7M -> unconnected-(J1-Pad36)
- J1 pad 37: /Connections/Q3 -> unconnected-(J1-Pad37)
- J1 pad 38: /Connections/PHI1 -> unconnected-(J1-Pad38)
