File: VGA-card/MPF-II_bus_adapter/KiCAD_prj/mpf-ii-bus-adapter.kicad_sch (KiCad schematic)
At the start: 11 parts, among them J1 Bus_Apple_II_Card_Side, J2 Bus_Apple_II_Computer_Side, J3 DevSel_Sel, J4 Phi0_Sel, J5 -12V_Selection, U1 74LS04

Commit message: Schematics updated
Parts:
- added J10: USER1_Sel, Connector_PinHeader_2.54mm:PinHeader_1x02_P2.54mm_Vertical, symbol Connector:Conn_01x02_Pin
- added J11: INH_Sel, Connector_PinHeader_2.54mm:PinHeader_1x02_P2.54mm_Vertical, symbol Connector:Conn_01x02_Pin
- added J12: RDY_Sel, Connector_PinHeader_2.54mm:PinHeader_1x02_P2.54mm_Vertical, symbol Connector:Conn_01x02_Pin
- added J13: COLREF_Sel, Connector_PinHeader_2.54mm:PinHeader_1x02_P2.54mm_Vertical, symbol Connector:Conn_01x02_Pin
- added J14: IOSTRB_Sel, Connector_PinHeader_2.54mm:PinHeader_1x02_P2.54mm_Vertical, symbol Connector:Conn_01x02_Pin
- added J15: Q3_Sel, Connector_PinHeader_2.54mm:PinHeader_1x02_P2.54mm_Vertical, symbol Connector:Conn_01x02_Pin
- added J16, J17, J18, J19, J20, J21, J22, J23, J24, J25: Pin, Connector_PinHeader_2.00mm:PinHeader_1x01_P2.00mm_Vertical, symbol Connector:Conn_01x01_Pin
- added J26: 7M_Sel, Connector_PinHeader_2.54mm:PinHeader_1x02_P2.54mm_Vertical, symbol Connector:Conn_01x02_Pin
- added J6: SYNC_Sel, Connector_PinHeader_2.54mm:PinHeader_1x02_P2.54mm_Vertical, symbol Connector:Conn_01x02_Pin
- added J7: DMA_Sel, Connector_PinHeader_2.54mm:PinHeader_1x02_P2.54mm_Vertical, symbol Connector:Conn_01x02_Pin
- added J8: IRQ_Sel, Connector_PinHeader_2.54mm:PinHeader_1x02_P2.54mm_Vertical, symbol Connector:Conn_01x02_Pin
- added J9: NMI_Sel, Connector_PinHeader_2.54mm:PinHeader_1x02_P2.54mm_Vertical, symbol Connector:Conn_01x02_Pin
- J5: value -12V_Selection -> -12V_Sel
Connections:
- net at U1.10: now also J22.1 (Pin_1)
- net at U1.11: now also J19.1 (Pin_1)
- net at U1.5: now also J17.1 (Pin_1)
- net at U1.6: now also J24.1 (Pin_1)
- net SYNC: now reaches J2.19 (TESTPIN)
- net SYNC: now also J6.1 (Pin_1)
- net IOSTRB: now reaches J2.20 (~{I/O_STROBE})
- net IOSTRB: now also J14.2 (Pin_2)
- net A_RDY: now reaches J2.21 (RDY)
- net A_RDY: now also J12.1 (Pin_1)
- net A_DMA: now reaches J2.22 (~{DMA})
- net A_DMA: now also J7.1 (Pin_1)
- net INTOUT: now reaches J2.23 (INT_OUT)
- net INTOUT: now also J1.23 (INT_OUT)
- net DMAOUT: now reaches J2.24 (DMA_OUT)
- net DMAOUT: now also J1.24 (DMA_OUT)
- net INTIN: now reaches J2.28 (INT_IN)
- net INTIN: now also J1.28 (INT_IN)
- net A_NMI: now reaches J2.29 (~{NMI})
- net A_NMI: now also J9.1 (Pin_1)
- net A_IRQ: now reaches J2.30 (~{IRQ})
- net A_IRQ: now also J8.1 (Pin_1)
- net A_INH: now reaches J2.32 (~{INH})
- net A_INH: now also J11.1 (Pin_1)
- net COLORREF: now reaches J2.35 (TESTPIN)
- net COLORREF: now also J13.2 (Pin_2)
- net 7M: now reaches J2.36 (7M)
- net 7M: now also J26.2 (Pin_2)
- net Q3: now reaches J2.37 (Q3)
- net Q3: now also J15.1 (Pin_1)
- net A_USER1: now reaches J2.39 (USER1)
- net A_USER1: now also J10.1 (Pin_1)
- net EXT8: now reaches J1.19 (TESTPIN)
- net EXT8: now also J6.2 (Pin_2)
- net EXTE: now reaches J1.20 (~{I/O_STROBE})
- net EXTE: now also J14.1 (Pin_1)
- net M_RDY: now reaches J1.21 (RDY)
- net M_RDY: now also J12.2 (Pin_2)
- net M_DMA: now reaches J1.22 (~{DMA})
- net M_DMA: now also J7.2 (Pin_2)
- net M_NMI: now reaches J1.29 (~{NMI})
- net M_NMI: now also J9.2 (Pin_2)
- net M_IRQ: now reaches J1.30 (~{IRQ})
- net M_IRQ: now also J8.2 (Pin_2)
- net M_INH: now reaches J1.32 (~{INH})
- net M_INH: now also J11.2 (Pin_2)
- net EXT6: now reaches J1.35 (TESTPIN)
- net EXT6: now also J13.1 (Pin_1)
- net SOUND_IN: now reaches J1.36 (7M)
- net SOUND_IN: now also J26.1 (Pin_1)
- net 2M: now reaches J1.37 (Q3)
- net 2M: now also J15.2 (Pin_2)
- net M_USER1: now reaches J1.39 (USER1)
- net M_USER1: now also J10.2 (Pin_2)
- net at U1.12: now also J21.1 (Pin_1)
- net at U1.13: now also J20.1 (Pin_1)
- net at U1.8: now also J23.1 (Pin_1)
- net at U1.9: now also J18.1 (Pin_1)
- net at U1.3: now also J16.1 (Pin_1)
- net at U1.4: now also J25.1 (Pin_1)
Other:
- moved on the sheet: U1B, U1C, U1D, U1E, U1F
