File: VGA-card/MPF-II_vga_card/KiCAD_prj/mpf_ii_vga_card.kicad_sch (KiCad schematic)
At the start: 6 parts, among them J1 AppleBus, U1 74LVC245, U2 74LVC245, U3 74LVC245, U4 74LVC245, U5 Pico

Commit message: Sch updated
Parts:
- added J2: GPIO10_CFG, Connector_PinHeader_2.54mm:PinHeader_1x04_P2.54mm_Vertical, symbol Connector:Conn_01x04_Pin
Connections:
- net GND: now also J2.4 (Pin_4); no longer U3.1 (A->B)
- net S1: now reaches U4.2 (A0)
- net S1: now also U5.12 (GPIO9)
- net S2: now reaches U4.3 (A1)
- net S2: now also U5.11 (GPIO8)
- net at U4.5 (A3): now also J2.1 (Pin_1)
- net S3: now reaches U5.14 (GPIO10)
- net S3: now also J2.2 (Pin_2)
- new net: J2.3 (Pin_3), U3.1 (A->B)
- no-connect marks 16 -> 19
Other:
- note added: "(this is how the Rev A schematic was connected)"
- note added: "J2 configures GPIO10 behavior:"
- note added: "When 1+2 and 3+4 are bridged (the default)"
- note added: "When only 2+3 is bridged then GPIO10 should"
- note added: "You probably don't want to change it"
- note added: "be set as an output to control U3 direction"
- note added: "the video SYNC signal from the bus"
- note added: "then GPIO10 should be set as an input to read"
- moved on the sheet: U4

Commit message: Card schematics updated
Parts:
- added R1, R2, R3, R4: 10K, symbol Device:R
Connections:
- net +3.3V: now also U5.36 (3V3), R1.1, R2.1, R3.1
- net +5V: now also R4.1
- net DEVSEL: now also U4.17 (B1)
- net GND: now also U4.1 (A->B)
- net PHI0: now also U4.16 (B2)
- net RW: now also U4.18 (B0)
- net SYNC: now also U4.15 (B3), R4.2
- net at U3.19 (CE): now also U5.15 (GPIO11), R3.2
- net at U2.19 (CE): now also U5.16 (GPIO12), R2.2
- net at U5.17 (GPIO13): now also U1.19 (CE), R1.2

Commit message: VGA card schematics updated
Parts:
- added R5, R6, R7, R8: 1K, symbol Device:R
Connections:
- net GND: now also U4.19 (CE), R5.2, R6.2, R7.2, R8.2
- net at U4.11 (B7): now also R8.1
- net at U4.12 (B6): now also R7.1
- net at U4.13 (B5): now also R6.1
- net at U4.14 (B4): now also R5.1
- net PHI0_3.3: now reaches U4.4 (A2)
- no-connect marks 19 -> 23
